File: SmartChessHardware/SmartChessHardware.kicad_pcb (KiCad board)
At the start: 2 copper layers, 0 parts

Commit message: Worked on PCB
Parts:
- added C1: 100uF, Capacitor_SMD:C_0603_1608Metric, F.Cu at (-252.6, 301.9)
- added C100: 100nF, Capacitor_SMD:C_0603_1608Metric, F.Cu at (-68.2, 189.5)
- added C101: 100nF, Capacitor_SMD:C_0603_1608Metric, F.Cu at (-68.2, 192.0)
- added C102: 100nF, Capacitor_SMD:C_0603_1608Metric, F.Cu at (-68.2, 194.5)
- added C103: 100nF, Capacitor_SMD:C_0603_1608Metric, F.Cu at (-68.2, 197.0)
- added C104: 100nF, Capacitor_SMD:C_0603_1608Metric, F.Cu at (-68.2, 199.6)
- added C105: 100nF, Capacitor_SMD:C_0603_1608Metric, F.Cu at (-68.2, 202.1)
- added C106: 100nF, Capacitor_SMD:C_0603_1608Metric, F.Cu at (-68.2, 204.6)
- added C107: 100nF, Capacitor_SMD:C_0603_1608Metric, F.Cu at (-68.2, 207.1)
- added C108: 100nF, Capacitor_SMD:C_0603_1608Metric, F.Cu at (-68.2, 209.6)
- added C109: 100nF, Capacitor_SMD:C_0603_1608Metric, F.Cu at (-68.2, 212.1)
- added C110: 100nF, Capacitor_SMD:C_0603_1608Metric, F.Cu at (-68.2, 214.6)
- added C111: 100nF, Capacitor_SMD:C_0603_1608Metric, F.Cu at (-64.2, 189.5)
- added C112: 100nF, Capacitor_SMD:C_0603_1608Metric, F.Cu at (-64.2, 192.0)
- added C113: 100nF, Capacitor_SMD:C_0603_1608Metric, F.Cu at (-64.2, 194.5)
- added C114: 100uF, Capacitor_SMD:C_0603_1608Metric, F.Cu at (-64.2, 197.0)
- added C115: 100nF, Capacitor_SMD:C_0603_1608Metric, F.Cu at (-64.2, 199.6)
- added C116: 100nF, Capacitor_SMD:C_0603_1608Metric, F.Cu at (-64.2, 202.1)
- added C117: 100nF, Capacitor_SMD:C_0603_1608Metric, F.Cu at (-64.2, 204.6)
- added C118: 100nF, Capacitor_SMD:C_0603_1608Metric, F.Cu at (-64.2, 207.1)
- added C119: 100nF, Capacitor_SMD:C_0603_1608Metric, F.Cu at (-64.2, 209.6)
- added C120: 100nF, Capacitor_SMD:C_0603_1608Metric, F.Cu at (-64.2, 212.1)
- added C121: 100nF, Capacitor_SMD:C_0603_1608Metric, F.Cu at (-64.2, 214.6)
- added C122: 100nF, Capacitor_SMD:C_0603_1608Metric, F.Cu at (-60.2, 189.5)
- added C123: 100nF, Capacitor_SMD:C_0603_1608Metric, F.Cu at (-60.2, 192.0)
- added C124: 100nF, Capacitor_SMD:C_0603_1608Metric, F.Cu at (-60.2, 194.5)
- added C125: 100nF, Capacitor_SMD:C_0603_1608Metric, F.Cu at (-60.2, 197.0)
- added C126: 100nF, Capacitor_SMD:C_0603_1608Metric, F.Cu at (-60.2, 199.6)
- added C127: 100nF, Capacitor_SMD:C_0603_1608Metric, F.Cu at (-60.2, 202.1)
- added C128: 100nF, Capacitor_SMD:C_0603_1608Metric, F.Cu at (-60.2, 204.6)
- added C129: 100nF, Capacitor_SMD:C_0603_1608Metric, F.Cu at (-60.2, 207.1)
- added C130: 100nF, Capacitor_SMD:C_0603_1608Metric, F.Cu at (-60.2, 209.6)
- added C131: 100nF, Capacitor_SMD:C_0603_1608Metric, F.Cu at (-60.2, 212.1)
- added C132: 100nF, Capacitor_SMD:C_0603_1608Metric, F.Cu at (-60.2, 214.6)
- added C133: 100nF, Capacitor_SMD:C_0603_1608Metric, F.Cu at (-56.2, 189.5)
- added C134: 100nF, Capacitor_SMD:C_0603_1608Metric, F.Cu at (-56.2, 192.0)
- added C135: 100nF, Capacitor_SMD:C_0603_1608Metric, F.Cu at (-56.2, 194.5)
- added C136: 100nF, Capacitor_SMD:C_0603_1608Metric, F.Cu at (-56.2, 197.0)
- added C137: 100nF, Capacitor_SMD:C_0603_1608Metric, F.Cu at (-56.2, 199.6)
- added C138: 100nF, Capacitor_SMD:C_0603_1608Metric, F.Cu at (-56.2, 202.1)
- added C139: 100nF, Capacitor_SMD:C_0603_1608Metric, F.Cu at (-56.2, 204.6)
- added C140: 100nF, Capacitor_SMD:C_0603_1608Metric, F.Cu at (-56.2, 207.1)
- added C141: 100nF, Capacitor_SMD:C_0603_1608Metric, F.Cu at (-56.2, 209.6)
- added C142: 100nF, Capacitor_SMD:C_0603_1608Metric, F.Cu at (-56.2, 212.1)
- added C143: 100nF, Capacitor_SMD:C_0603_1608Metric, F.Cu at (-56.2, 214.6)
- added C144: 100nF, Capacitor_SMD:C_0603_1608Metric, F.Cu at (-52.2, 189.5)
- added C145: 100nF, Capacitor_SMD:C_0603_1608Metric, F.Cu at (-52.2, 192.0)
- added C146: 100nF, Capacitor_SMD:C_0603_1608Metric, F.Cu at (-52.2, 194.5)
- added C147: 100nF, Capacitor_SMD:C_0603_1608Metric, F.Cu at (-52.2, 197.0)
- added C148: 100nF, Capacitor_SMD:C_0603_1608Metric, F.Cu at (-52.2, 199.6)
- added C149: 100nF, Capacitor_SMD:C_0603_1608Metric, F.Cu at (-52.2, 202.1)
- added C150: 100nF, Capacitor_SMD:C_0603_1608Metric, F.Cu at (-52.2, 204.6)
- added C151: 100nF, Capacitor_SMD:C_0603_1608Metric, F.Cu at (-52.2, 207.1)
- added C152: 100nF, Capacitor_SMD:C_0603_1608Metric, F.Cu at (-52.2, 209.6)
- added C153: 100nF, Capacitor_SMD:C_0603_1608Metric, F.Cu at (-52.2, 212.1)
- added C154: 100nF, Capacitor_SMD:C_0603_1608Metric, F.Cu at (-52.2, 214.6)
- added C155: 100nF, Capacitor_SMD:C_0603_1608Metric, F.Cu at (-48.1, 189.5)
- added C156: 100nF, Capacitor_SMD:C_0603_1608Metric, F.Cu at (-48.1, 192.0)
- added C157: 100nF, Capacitor_SMD:C_0603_1608Metric, F.Cu at (-48.1, 194.5)
- added C158: 100nF, Capacitor_SMD:C_0603_1608Metric, F.Cu at (-48.1, 197.0)
- added C159: 100nF, Capacitor_SMD:C_0603_1608Metric, F.Cu at (-48.1, 199.6)
- added C160: 100nF, Capacitor_SMD:C_0603_1608Metric, F.Cu at (-48.1, 202.1)
- added C161: 100nF, Capacitor_SMD:C_0603_1608Metric, F.Cu at (-48.1, 204.6)
- added C162: 100nF, Capacitor_SMD:C_0603_1608Metric, F.Cu at (-48.1, 207.1)
- added C163: 100nF, Capacitor_SMD:C_0603_1608Metric, F.Cu at (-48.1, 209.6)
- added C164: 100nF, Capacitor_SMD:C_0603_1608Metric, F.Cu at (-48.1, 212.1)
- added C2: 100n, Capacitor_SMD:C_0603_1608Metric, F.Cu at (-252.6, 304.5)
- added C3: 100n, Capacitor_SMD:C_0603_1608Metric, F.Cu at (-252.6, 307.0)
- added C4: 100n, Capacitor_SMD:C_0603_1608Metric, F.Cu at (-252.6, 309.5)
- added D100: WS2812B, LED_SMD:LED_WS2812B_PLCC4_5.0x5.0mm_P3.2mm, F.Cu at (92.0, 34.0)
- added D101: WS2812B, LED_SMD:LED_WS2812B_PLCC4_5.0x5.0mm_P3.2mm, F.Cu at (122.0, 33.9)
- added D102: WS2812B, LED_SMD:LED_WS2812B_PLCC4_5.0x5.0mm_P3.2mm, F.Cu at (152.0, 33.5)
- added D103: WS2812B, LED_SMD:LED_WS2812B_PLCC4_5.0x5.0mm_P3.2mm, F.Cu at (182.0, 33.5)
- added D104: WS2812B, LED_SMD:LED_WS2812B_PLCC4_5.0x5.0mm_P3.2mm, F.Cu at (212.0, 33.5)
- added D105: WS2812B, LED_SMD:LED_WS2812B_PLCC4_5.0x5.0mm_P3.2mm, F.Cu at (242.0, 33.5)
- added D106: WS2812B, LED_SMD:LED_WS2812B_PLCC4_5.0x5.0mm_P3.2mm, F.Cu at (272.0, 34.1)
- added D107: WS2812B, LED_SMD:LED_WS2812B_PLCC4_5.0x5.0mm_P3.2mm, F.Cu at (302.0, 34.0)
- added D108: WS2812B, LED_SMD:LED_WS2812B_PLCC4_5.0x5.0mm_P3.2mm, F.Cu at (-58.0, 138.6)
- added D109: WS2812B, LED_SMD:LED_WS2812B_PLCC4_5.0x5.0mm_P3.2mm, F.Cu at (-58.0, 145.2)
- added D110: WS2812B, LED_SMD:LED_WS2812B_PLCC4_5.0x5.0mm_P3.2mm, F.Cu at (-58.0, 151.8)
- added D111: WS2812B, LED_SMD:LED_WS2812B_PLCC4_5.0x5.0mm_P3.2mm, F.Cu at (-58.0, 158.5)
- added D112: WS2812B, LED_SMD:LED_WS2812B_PLCC4_5.0x5.0mm_P3.2mm, F.Cu at (-58.0, 165.1)
- added D113: WS2812B, LED_SMD:LED_WS2812B_PLCC4_5.0x5.0mm_P3.2mm, F.Cu at (-58.0, 171.7)
- added D114: WS2812B, LED_SMD:LED_WS2812B_PLCC4_5.0x5.0mm_P3.2mm, F.Cu at (-58.0, 178.3)
- added D115: WS2812B, LED_SMD:LED_WS2812B_PLCC4_5.0x5.0mm_P3.2mm, F.Cu at (-58.0, 184.9)
- added D116: WS2812B, LED_SMD:LED_WS2812B_PLCC4_5.0x5.0mm_P3.2mm, F.Cu at (-49.9, 138.6)
- added D117: WS2812B, LED_SMD:LED_WS2812B_PLCC4_5.0x5.0mm_P3.2mm, F.Cu at (-49.9, 145.2)
- added D118: WS2812B, LED_SMD:LED_WS2812B_PLCC4_5.0x5.0mm_P3.2mm, F.Cu at (-49.9, 151.8)
- added D119: WS2812B, LED_SMD:LED_WS2812B_PLCC4_5.0x5.0mm_P3.2mm, F.Cu at (-49.9, 158.5)
- added D120: WS2812B, LED_SMD:LED_WS2812B_PLCC4_5.0x5.0mm_P3.2mm, F.Cu at (-49.9, 165.1)
- added D121: WS2812B, LED_SMD:LED_WS2812B_PLCC4_5.0x5.0mm_P3.2mm, F.Cu at (-49.9, 171.7)
- added D122: WS2812B, LED_SMD:LED_WS2812B_PLCC4_5.0x5.0mm_P3.2mm, F.Cu at (-49.9, 178.3)
- added D123: WS2812B, LED_SMD:LED_WS2812B_PLCC4_5.0x5.0mm_P3.2mm, F.Cu at (-49.9, 184.9)
- added D124: WS2812B, LED_SMD:LED_WS2812B_PLCC4_5.0x5.0mm_P3.2mm, F.Cu at (-41.8, 138.6)
- added D125: WS2812B, LED_SMD:LED_WS2812B_PLCC4_5.0x5.0mm_P3.2mm, F.Cu at (-41.8, 145.2)
- added D126: WS2812B, LED_SMD:LED_WS2812B_PLCC4_5.0x5.0mm_P3.2mm, F.Cu at (-41.8, 151.8)
- added D127: WS2812B, LED_SMD:LED_WS2812B_PLCC4_5.0x5.0mm_P3.2mm, F.Cu at (-41.8, 158.5)
- added D128: WS2812B, LED_SMD:LED_WS2812B_PLCC4_5.0x5.0mm_P3.2mm, F.Cu at (-41.8, 165.1)
- added D129: WS2812B, LED_SMD:LED_WS2812B_PLCC4_5.0x5.0mm_P3.2mm, F.Cu at (-41.8, 171.7)
- added D130: WS2812B, LED_SMD:LED_WS2812B_PLCC4_5.0x5.0mm_P3.2mm, F.Cu at (-41.8, 178.3)
- added D131: WS2812B, LED_SMD:LED_WS2812B_PLCC4_5.0x5.0mm_P3.2mm, F.Cu at (-41.8, 184.9)
- added D132: WS2812B, LED_SMD:LED_WS2812B_PLCC4_5.0x5.0mm_P3.2mm, F.Cu at (-33.7, 138.6)
- added D133: WS2812B, LED_SMD:LED_WS2812B_PLCC4_5.0x5.0mm_P3.2mm, F.Cu at (-33.7, 145.2)
- added D134: WS2812B, LED_SMD:LED_WS2812B_PLCC4_5.0x5.0mm_P3.2mm, F.Cu at (-33.7, 151.8)
- added D135: WS2812B, LED_SMD:LED_WS2812B_PLCC4_5.0x5.0mm_P3.2mm, F.Cu at (-33.7, 158.5)
- added D136: WS2812B, LED_SMD:LED_WS2812B_PLCC4_5.0x5.0mm_P3.2mm, F.Cu at (-33.7, 165.1)
- added D137: WS2812B, LED_SMD:LED_WS2812B_PLCC4_5.0x5.0mm_P3.2mm, F.Cu at (-33.7, 171.7)
- added D138: WS2812B, LED_SMD:LED_WS2812B_PLCC4_5.0x5.0mm_P3.2mm, F.Cu at (-33.7, 178.3)
- added D139: WS2812B, LED_SMD:LED_WS2812B_PLCC4_5.0x5.0mm_P3.2mm, F.Cu at (-33.7, 184.9)
- added D140: WS2812B, LED_SMD:LED_WS2812B_PLCC4_5.0x5.0mm_P3.2mm, F.Cu at (-25.5, 138.6)
- added D141: WS2812B, LED_SMD:LED_WS2812B_PLCC4_5.0x5.0mm_P3.2mm, F.Cu at (-25.5, 145.2)
- added D142: WS2812B, LED_SMD:LED_WS2812B_PLCC4_5.0x5.0mm_P3.2mm, F.Cu at (-25.5, 151.8)
- added D143: WS2812B, LED_SMD:LED_WS2812B_PLCC4_5.0x5.0mm_P3.2mm, F.Cu at (-25.5, 158.5)
- added D144: WS2812B, LED_SMD:LED_WS2812B_PLCC4_5.0x5.0mm_P3.2mm, F.Cu at (-25.5, 165.1)
- added D145: WS2812B, LED_SMD:LED_WS2812B_PLCC4_5.0x5.0mm_P3.2mm, F.Cu at (-25.5, 171.7)
- added D146: WS2812B, LED_SMD:LED_WS2812B_PLCC4_5.0x5.0mm_P3.2mm, F.Cu at (-25.5, 178.3)
- added D147: WS2812B, LED_SMD:LED_WS2812B_PLCC4_5.0x5.0mm_P3.2mm, F.Cu at (-25.5, 184.9)
- added D148: WS2812B, LED_SMD:LED_WS2812B_PLCC4_5.0x5.0mm_P3.2mm, F.Cu at (-17.4, 138.6)
- added D149: WS2812B, LED_SMD:LED_WS2812B_PLCC4_5.0x5.0mm_P3.2mm, F.Cu at (-17.4, 145.2)
- added D150: WS2812B, LED_SMD:LED_WS2812B_PLCC4_5.0x5.0mm_P3.2mm, F.Cu at (-17.4, 151.8)
- added D151: WS2812B, LED_SMD:LED_WS2812B_PLCC4_5.0x5.0mm_P3.2mm, F.Cu at (-17.4, 158.5)
- added D152: WS2812B, LED_SMD:LED_WS2812B_PLCC4_5.0x5.0mm_P3.2mm, F.Cu at (-17.4, 165.1)
- added D153: WS2812B, LED_SMD:LED_WS2812B_PLCC4_5.0x5.0mm_P3.2mm, F.Cu at (-17.4, 171.7)
- added D154: WS2812B, LED_SMD:LED_WS2812B_PLCC4_5.0x5.0mm_P3.2mm, F.Cu at (-17.4, 178.3)
- added D155: WS2812B, LED_SMD:LED_WS2812B_PLCC4_5.0x5.0mm_P3.2mm, F.Cu at (-17.4, 184.9)
- added D156: WS2812B, LED_SMD:LED_WS2812B_PLCC4_5.0x5.0mm_P3.2mm, F.Cu at (-9.30, 138.6)
- added D157: WS2812B, LED_SMD:LED_WS2812B_PLCC4_5.0x5.0mm_P3.2mm, F.Cu at (-9.30, 145.2)
- added D158: WS2812B, LED_SMD:LED_WS2812B_PLCC4_5.0x5.0mm_P3.2mm, F.Cu at (-9.30, 151.8)
- added D159: WS2812B, LED_SMD:LED_WS2812B_PLCC4_5.0x5.0mm_P3.2mm, F.Cu at (-9.30, 158.5)
- added D160: WS2812B, LED_SMD:LED_WS2812B_PLCC4_5.0x5.0mm_P3.2mm, F.Cu at (-9.30, 165.1)
- added D161: WS2812B, LED_SMD:LED_WS2812B_PLCC4_5.0x5.0mm_P3.2mm, F.Cu at (-9.30, 171.7)
- added D162: WS2812B, LED_SMD:LED_WS2812B_PLCC4_5.0x5.0mm_P3.2mm, F.Cu at (-9.30, 178.3)
- added D163: WS2812B, LED_SMD:LED_WS2812B_PLCC4_5.0x5.0mm_P3.2mm, F.Cu at (-9.30, 184.9)
- added D200: 1N4001, Diode_SMD:D_SMA, F.Cu at (82.0, 49.0)
- added D201: 1N4001, Diode_SMD:D_SMA, F.Cu at (111.5, 48.5)
- added D202: 1N4001, Diode_SMD:D_SMA, F.Cu at (141.5, 48.5)
- added D203: 1N4001, Diode_SMD:D_SMA, F.Cu at (172.0, 49.5)
- added D204: 1N4001, Diode_SMD:D_SMA, F.Cu at (202.5, 50.5)
- added D205: 1N4001, Diode_SMD:D_SMA, F.Cu at (235.5, 51.0)
- added D206: 1N4001, Diode_SMD:D_SMA, F.Cu at (263.5, 50.0)
- added D207: 1N4001, Diode_SMD:D_SMA, F.Cu at (292.0, 52.5)
- added D208: 1N4001, Diode_SMD:D_SMA, F.Cu at (-66.1, 121.9)
- added D209: 1N4001, Diode_SMD:D_SMA, F.Cu at (-66.1, 126.5)
- added D210: 1N4001, Diode_SMD:D_SMA, F.Cu at (-66.1, 131.0)
- added D211: 1N4001, Diode_SMD:D_SMA, F.Cu at (-58.0, 85.5)
- added D212: 1N4001, Diode_SMD:D_SMA, F.Cu at (-58.0, 90.1)
- added D213: 1N4001, Diode_SMD:D_SMA, F.Cu at (-58.0, 94.6)
- added D214: 1N4001, Diode_SMD:D_SMA, F.Cu at (-58.0, 99.2)
- added D215: 1N4001, Diode_SMD:D_SMA, F.Cu at (-58.0, 103.7)
- added D216: 1N4001, Diode_SMD:D_SMA, F.Cu at (-58.0, 108.3)
- added D217: 1N4001, Diode_SMD:D_SMA, F.Cu at (-58.0, 112.8)
- added D218: 1N4001, Diode_SMD:D_SMA, F.Cu at (-58.0, 117.4)
- added D219: 1N4001, Diode_SMD:D_SMA, F.Cu at (-58.0, 121.9)
- added D220: 1N4001, Diode_SMD:D_SMA, F.Cu at (-58.0, 126.5)
- added D221: 1N4001, Diode_SMD:D_SMA, F.Cu at (-58.0, 131.0)
- added D222: 1N4001, Diode_SMD:D_SMA, F.Cu at (-49.9, 85.5)
- added D223: 1N4001, Diode_SMD:D_SMA, F.Cu at (-49.9, 90.1)
- added D224: 1N4001, Diode_SMD:D_SMA, F.Cu at (-49.9, 94.6)
- added D225: 1N4001, Diode_SMD:D_SMA, F.Cu at (-49.9, 99.2)
- added D226: 1N4001, Diode_SMD:D_SMA, F.Cu at (-49.9, 103.7)
- added D227: 1N4001, Diode_SMD:D_SMA, F.Cu at (-49.9, 108.3)
- added D228: 1N4001, Diode_SMD:D_SMA, F.Cu at (-49.9, 112.8)
- added D229: 1N4001, Diode_SMD:D_SMA, F.Cu at (-49.9, 117.4)
- added D230: 1N4001, Diode_SMD:D_SMA, F.Cu at (-49.9, 121.9)
- added D231: 1N4001, Diode_SMD:D_SMA, F.Cu at (-49.9, 126.5)
- added D232: 1N4001, Diode_SMD:D_SMA, F.Cu at (-49.9, 131.0)
- added D233: 1N4001, Diode_SMD:D_SMA, F.Cu at (-41.8, 85.5)
- added D234: 1N4001, Diode_SMD:D_SMA, F.Cu at (-41.8, 90.1)
- added D235: 1N4001, Diode_SMD:D_SMA, F.Cu at (-41.8, 94.6)
- added D236: 1N4001, Diode_SMD:D_SMA, F.Cu at (-41.8, 99.2)
- added D237: 1N4001, Diode_SMD:D_SMA, F.Cu at (-41.8, 103.7)
- added D238: 1N4001, Diode_SMD:D_SMA, F.Cu at (-41.8, 108.3)
- added D239: 1N4001, Diode_SMD:D_SMA, F.Cu at (-41.8, 112.8)
- added D240: 1N4001, Diode_SMD:D_SMA, F.Cu at (-41.8, 117.4)
- added D241: 1N4001, Diode_SMD:D_SMA, F.Cu at (-41.8, 121.9)
- added D242: 1N4001, Diode_SMD:D_SMA, F.Cu at (-41.8, 126.5)
- added D243: 1N4001, Diode_SMD:D_SMA, F.Cu at (-41.8, 131.0)
- added D244: 1N4001, Diode_SMD:D_SMA, F.Cu at (-33.8, 85.5)
- added D245: 1N4001, Diode_SMD:D_SMA, F.Cu at (-33.8, 90.1)
- added D246: 1N4001, Diode_SMD:D_SMA, F.Cu at (-33.8, 94.6)
- added D247: 1N4001, Diode_SMD:D_SMA, F.Cu at (-33.8, 99.2)
- added D248: 1N4001, Diode_SMD:D_SMA, F.Cu at (-33.8, 103.7)
- added D249: 1N4001, Diode_SMD:D_SMA, F.Cu at (-33.8, 108.3)
- added D250: 1N4001, Diode_SMD:D_SMA, F.Cu at (-33.8, 112.8)
- added D251: 1N4001, Diode_SMD:D_SMA, F.Cu at (-33.8, 117.4)
- added D252: 1N4001, Diode_SMD:D_SMA, F.Cu at (-33.8, 121.9)
- added D253: 1N4001, Diode_SMD:D_SMA, F.Cu at (-33.8, 126.5)
- added D254: 1N4001, Diode_SMD:D_SMA, F.Cu at (-33.8, 131.0)
- added D255: 1N4001, Diode_SMD:D_SMA, F.Cu at (-25.7, 85.5)
- added D256: 1N4001, Diode_SMD:D_SMA, F.Cu at (-25.7, 90.1)
- added D257: 1N4001, Diode_SMD:D_SMA, F.Cu at (-25.7, 94.6)
- added D258: 1N4001, Diode_SMD:D_SMA, F.Cu at (-25.7, 99.2)
- added D259: 1N4001, Diode_SMD:D_SMA, F.Cu at (-25.7, 103.7)
- added D260: 1N4001, Diode_SMD:D_SMA, F.Cu at (-25.7, 108.3)
- added D261: 1N4001, Diode_SMD:D_SMA, F.Cu at (-25.7, 112.8)
- added D262: 1N4001, Diode_SMD:D_SMA, F.Cu at (-25.7, 117.4)
- added D263: 1N4001, Diode_SMD:D_SMA, F.Cu at (-25.7, 121.9)
- added F1: 10A, Fuse:Fuse_0603_1608Metric, F.Cu at (-252.6, 312.0)
- added IC1: Pi-Zero-UART, Module:Raspberry_Pi_Zero_Socketed_THT_FaceDown_MountingHoles, F.Cu at (-308.0, 254.9)
- added IC2: Arduino_UNO_R3, Module:Arduino_UNO_R3, F.Cu at (-244.8, 249.1)
- added IC3: MCP23017x-x-SO, Package_SO:SOIC-28W_7.5x17.9mm_P1.27mm, F.Cu at (-273.4, 310.5)
- added J1: Barrel_Jack, Connector_BarrelJack:BarrelJack_GCT_DCJ200-10-A_Horizontal, F.Cu at (-261.5, 302.7)
- added JP1: Jumper_2_Open, Connector_PinHeader_1.00mm:PinHeader_1x02_P1.00mm_Vertical, F.Cu at (-228.8, 302.2)
- added JP2: Jumper_2_Open, Connector_PinHeader_1.00mm:PinHeader_1x02_P1.00mm_Vertical, F.Cu at (-225.4, 302.2)
- added JP3: Jumper_2_Open, Connector_PinHeader_1.00mm:PinHeader_1x02_P1.00mm_Vertical, F.Cu at (-222.1, 302.2)
- added JP4: Jumper UART Pi -> Arduino, Connector_PinHeader_1.00mm:PinHeader_1x02_P1.00mm_Vertical, F.Cu at (-218.8, 302.2)
- added JP5: Jumper UART Arduino -> Pi, Connector_PinHeader_1.00mm:PinHeader_1x02_P1.00mm_Vertical, F.Cu at (-215.4, 302.2)
- added Print200: ChessboardPrint, SmartChessCustomFootprints:ChessBoard, F.Cu at (77.0, 27.9)
- added R1: 220R, Resistor_SMD:R_0603_1608Metric, F.Cu at (-252.6, 314.5)
- added R2: 5,2K, Resistor_SMD:R_0603_1608Metric, F.Cu at (-248.6, 301.9)
- added R200: 10K, Resistor_SMD:R_0603_1608Metric, F.Cu at (-19.6, 84.5)
- added R201: 10K, Resistor_SMD:R_0603_1608Metric, F.Cu at (-19.6, 87.0)
- added R202: 10K, Resistor_SMD:R_0603_1608Metric, F.Cu at (-19.6, 89.5)
- added R203: 10K, Resistor_SMD:R_0603_1608Metric, F.Cu at (-19.6, 92.0)
- added R204: 10K, Resistor_SMD:R_0603_1608Metric, F.Cu at (-19.6, 94.5)
- added R205: 10K, Resistor_SMD:R_0603_1608Metric, F.Cu at (-19.6, 97.1)
- added R206: 10K, Resistor_SMD:R_0603_1608Metric, F.Cu at (-19.6, 99.6)
- added R207: 10K, Resistor_SMD:R_0603_1608Metric, F.Cu at (-19.6, 102.1)
- added R3: 10K, Resistor_SMD:R_0603_1608Metric, F.Cu at (-248.6, 304.5)
- added R4: 10K, Resistor_SMD:R_0603_1608Metric, F.Cu at (-248.6, 307.0)
- added R5: 10K, Resistor_SMD:R_0603_1608Metric, F.Cu at (-248.6, 309.5)
- added R6: 10k, Resistor_SMD:R_0603_1608Metric, F.Cu at (-248.6, 312.0)
- added SW200: SW_Reed, Resistor_THT:R_Axial_DIN0309_L9.0mm_D3.2mm_P20.32mm_Horizontal, F.Cu at (81.8, 42.0)
- added SW201: SW_Reed, Resistor_THT:R_Axial_DIN0309_L9.0mm_D3.2mm_P20.32mm_Horizontal, F.Cu at (111.7, 42.0)
- added SW202: SW_Reed, Resistor_THT:R_Axial_DIN0309_L9.0mm_D3.2mm_P20.32mm_Horizontal, F.Cu at (141.7, 41.5)
- added SW203: SW_Reed, Resistor_THT:R_Axial_DIN0309_L9.0mm_D3.2mm_P20.32mm_Horizontal, F.Cu at (172.2, 43.5)
- added SW204: SW_Reed, Resistor_THT:R_Axial_DIN0309_L9.0mm_D3.2mm_P20.32mm_Horizontal, F.Cu at (201.7, 44.0)
- added SW205: SW_Reed, Resistor_THT:R_Axial_DIN0309_L9.0mm_D3.2mm_P20.32mm_Horizontal, F.Cu at (234.5, 43.0)
- added SW206: SW_Reed, Resistor_THT:R_Axial_DIN0309_L9.0mm_D3.2mm_P20.32mm_Horizontal, F.Cu at (263.0, 43.0)
- added SW207: SW_Reed, Resistor_THT:R_Axial_DIN0309_L9.0mm_D3.2mm_P20.32mm_Horizontal, F.Cu at (292.0, 43.5)
- added SW208: SW_Reed, Resistor_THT:R_Axial_DIN0309_L9.0mm_D3.2mm_P20.32mm_Horizontal, F.Cu at (-68.6, 42.9)
- added SW209: SW_Reed, Resistor_THT:R_Axial_DIN0309_L9.0mm_D3.2mm_P20.32mm_Horizontal, F.Cu at (-68.6, 47.6)
- added SW210: SW_Reed, Resistor_THT:R_Axial_DIN0309_L9.0mm_D3.2mm_P20.32mm_Horizontal, F.Cu at (-68.6, 52.4)
- added SW211: SW_Reed, Resistor_THT:R_Axial_DIN0309_L9.0mm_D3.2mm_P20.32mm_Horizontal, F.Cu at (-68.6, 57.1)
- added SW212: SW_Reed, Resistor_THT:R_Axial_DIN0309_L9.0mm_D3.2mm_P20.32mm_Horizontal, F.Cu at (-68.6, 61.9)
- added SW213: SW_Reed, Resistor_THT:R_Axial_DIN0309_L9.0mm_D3.2mm_P20.32mm_Horizontal, F.Cu at (-68.6, 66.6)
- added SW214: SW_Reed, Resistor_THT:R_Axial_DIN0309_L9.0mm_D3.2mm_P20.32mm_Horizontal, F.Cu at (-68.6, 71.4)
- added SW215: SW_Reed, Resistor_THT:R_Axial_DIN0309_L9.0mm_D3.2mm_P20.32mm_Horizontal, F.Cu at (-68.6, 76.1)
- added SW216: SW_Reed, Resistor_THT:R_Axial_DIN0309_L9.0mm_D3.2mm_P20.32mm_Horizontal, F.Cu at (-68.6, 80.9)
- added SW217: SW_Reed, Resistor_THT:R_Axial_DIN0309_L9.0mm_D3.2mm_P20.32mm_Horizontal, F.Cu at (-45.2, 4.88)
- added SW218: SW_Reed, Resistor_THT:R_Axial_DIN0309_L9.0mm_D3.2mm_P20.32mm_Horizontal, F.Cu at (-45.2, 9.62)
- added SW219: SW_Reed, Resistor_THT:R_Axial_DIN0309_L9.0mm_D3.2mm_P20.32mm_Horizontal, F.Cu at (-45.2, 14.4)
- added SW220: SW_Reed, Resistor_THT:R_Axial_DIN0309_L9.0mm_D3.2mm_P20.32mm_Horizontal, F.Cu at (-45.2, 19.1)
- added SW221: SW_Reed, Resistor_THT:R_Axial_DIN0309_L9.0mm_D3.2mm_P20.32mm_Horizontal, F.Cu at (-45.2, 23.9)
- added SW222: SW_Reed, Resistor_THT:R_Axial_DIN0309_L9.0mm_D3.2mm_P20.32mm_Horizontal, F.Cu at (-45.2, 28.6)
- added SW223: SW_Reed, Resistor_THT:R_Axial_DIN0309_L9.0mm_D3.2mm_P20.32mm_Horizontal, F.Cu at (-45.2, 33.4)
- added SW224: SW_Reed, Resistor_THT:R_Axial_DIN0309_L9.0mm_D3.2mm_P20.32mm_Horizontal, F.Cu at (-45.2, 38.1)
- added SW225: SW_Reed, Resistor_THT:R_Axial_DIN0309_L9.0mm_D3.2mm_P20.32mm_Horizontal, F.Cu at (-45.2, 42.9)
- added SW226: SW_Reed, Resistor_THT:R_Axial_DIN0309_L9.0mm_D3.2mm_P20.32mm_Horizontal, F.Cu at (-45.2, 47.6)
- added SW227: SW_Reed, Resistor_THT:R_Axial_DIN0309_L9.0mm_D3.2mm_P20.32mm_Horizontal, F.Cu at (-45.2, 52.4)
- added SW228: SW_Reed, Resistor_THT:R_Axial_DIN0309_L9.0mm_D3.2mm_P20.32mm_Horizontal, F.Cu at (-45.2, 57.1)
- added SW229: SW_Reed, Resistor_THT:R_Axial_DIN0309_L9.0mm_D3.2mm_P20.32mm_Horizontal, F.Cu at (-45.2, 61.9)
- added SW230: SW_Reed, Resistor_THT:R_Axial_DIN0309_L9.0mm_D3.2mm_P20.32mm_Horizontal, F.Cu at (-45.2, 66.6)
- added SW231: SW_Reed, Resistor_THT:R_Axial_DIN0309_L9.0mm_D3.2mm_P20.32mm_Horizontal, F.Cu at (-45.2, 71.4)
- added SW232: SW_Reed, Resistor_THT:R_Axial_DIN0309_L9.0mm_D3.2mm_P20.32mm_Horizontal, F.Cu at (-45.2, 76.1)
- added SW233: SW_Reed, Resistor_THT:R_Axial_DIN0309_L9.0mm_D3.2mm_P20.32mm_Horizontal, F.Cu at (-45.2, 80.9)
- added SW234: SW_Reed, Resistor_THT:R_Axial_DIN0309_L9.0mm_D3.2mm_P20.32mm_Horizontal, F.Cu at (-21.7, 4.88)
- added SW235: SW_Reed, Resistor_THT:R_Axial_DIN0309_L9.0mm_D3.2mm_P20.32mm_Horizontal, F.Cu at (-21.7, 9.62)
- added SW236: SW_Reed, Resistor_THT:R_Axial_DIN0309_L9.0mm_D3.2mm_P20.32mm_Horizontal, F.Cu at (-21.7, 14.4)
- added SW237: SW_Reed, Resistor_THT:R_Axial_DIN0309_L9.0mm_D3.2mm_P20.32mm_Horizontal, F.Cu at (-21.7, 19.1)
- added SW238: SW_Reed, Resistor_THT:R_Axial_DIN0309_L9.0mm_D3.2mm_P20.32mm_Horizontal, F.Cu at (-21.7, 23.9)
- added SW239: SW_Reed, Resistor_THT:R_Axial_DIN0309_L9.0mm_D3.2mm_P20.32mm_Horizontal, F.Cu at (-21.7, 28.6)
- added SW240: SW_Reed, Resistor_THT:R_Axial_DIN0309_L9.0mm_D3.2mm_P20.32mm_Horizontal, F.Cu at (-21.7, 33.4)
- added SW241: SW_Reed, Resistor_THT:R_Axial_DIN0309_L9.0mm_D3.2mm_P20.32mm_Horizontal, F.Cu at (-21.7, 38.1)
- added SW242: SW_Reed, Resistor_THT:R_Axial_DIN0309_L9.0mm_D3.2mm_P20.32mm_Horizontal, F.Cu at (-21.7, 42.9)
- added SW243: SW_Reed, Resistor_THT:R_Axial_DIN0309_L9.0mm_D3.2mm_P20.32mm_Horizontal, F.Cu at (-21.7, 47.6)
- added SW244: SW_Reed, Resistor_THT:R_Axial_DIN0309_L9.0mm_D3.2mm_P20.32mm_Horizontal, F.Cu at (-21.7, 52.4)
- added SW245: SW_Reed, Resistor_THT:R_Axial_DIN0309_L9.0mm_D3.2mm_P20.32mm_Horizontal, F.Cu at (-21.7, 57.1)
- added SW246: SW_Reed, Resistor_THT:R_Axial_DIN0309_L9.0mm_D3.2mm_P20.32mm_Horizontal, F.Cu at (-21.7, 61.9)
- added SW247: SW_Reed, Resistor_THT:R_Axial_DIN0309_L9.0mm_D3.2mm_P20.32mm_Horizontal, F.Cu at (-21.7, 66.6)
- added SW248: SW_Reed, Resistor_THT:R_Axial_DIN0309_L9.0mm_D3.2mm_P20.32mm_Horizontal, F.Cu at (-21.7, 71.4)
- added SW249: SW_Reed, Resistor_THT:R_Axial_DIN0309_L9.0mm_D3.2mm_P20.32mm_Horizontal, F.Cu at (-21.7, 76.1)
- added SW250: SW_Reed, Resistor_THT:R_Axial_DIN0309_L9.0mm_D3.2mm_P20.32mm_Horizontal, F.Cu at (-21.7, 80.9)
- added SW251: SW_Reed, Resistor_THT:R_Axial_DIN0309_L9.0mm_D3.2mm_P20.32mm_Horizontal, F.Cu at (1.78, 4.88)
- added SW252: SW_Reed, Resistor_THT:R_Axial_DIN0309_L9.0mm_D3.2mm_P20.32mm_Horizontal, F.Cu at (1.78, 9.62)
- added SW253: SW_Reed, Resistor_THT:R_Axial_DIN0309_L9.0mm_D3.2mm_P20.32mm_Horizontal, F.Cu at (1.78, 14.4)
- added SW254: SW_Reed, Resistor_THT:R_Axial_DIN0309_L9.0mm_D3.2mm_P20.32mm_Horizontal, F.Cu at (1.78, 19.1)
- added SW255: SW_Reed, Resistor_THT:R_Axial_DIN0309_L9.0mm_D3.2mm_P20.32mm_Horizontal, F.Cu at (1.78, 23.9)
- added SW256: SW_Reed, Resistor_THT:R_Axial_DIN0309_L9.0mm_D3.2mm_P20.32mm_Horizontal, F.Cu at (1.78, 28.6)
- added SW257: SW_Reed, Resistor_THT:R_Axial_DIN0309_L9.0mm_D3.2mm_P20.32mm_Horizontal, F.Cu at (1.78, 33.4)
- added SW258: SW_Reed, Resistor_THT:R_Axial_DIN0309_L9.0mm_D3.2mm_P20.32mm_Horizontal, F.Cu at (1.78, 38.1)
- added SW259: SW_Reed, Resistor_THT:R_Axial_DIN0309_L9.0mm_D3.2mm_P20.32mm_Horizontal, F.Cu at (1.78, 42.9)
- added SW260: SW_Reed, Resistor_THT:R_Axial_DIN0309_L9.0mm_D3.2mm_P20.32mm_Horizontal, F.Cu at (1.78, 47.6)
- added SW261: SW_Reed, Resistor_THT:R_Axial_DIN0309_L9.0mm_D3.2mm_P20.32mm_Horizontal, F.Cu at (1.78, 52.4)
- added SW262: SW_Reed, Resistor_THT:R_Axial_DIN0309_L9.0mm_D3.2mm_P20.32mm_Horizontal, F.Cu at (1.78, 57.1)
- added SW263: SW_Reed, Resistor_THT:R_Axial_DIN0309_L9.0mm_D3.2mm_P20.32mm_Horizontal, F.Cu at (1.78, 61.9)
- added TP1: GND, TestPoint:TestPoint_THTPad_D2.0mm_Drill1.0mm, F.Cu at (-244.6, 302.7)
- added TP2: +5V, TestPoint:TestPoint_THTPad_D2.0mm_Drill1.0mm, F.Cu at (-244.6, 306.8)
- added TP3: UART Arduino -> PI (5V), TestPoint:TestPoint_THTPad_D2.0mm_Drill1.0mm, F.Cu at (-240.5, 302.7)
- added TP4: UART PI -> Arduino, TestPoint:TestPoint_THTPad_D2.0mm_Drill1.0mm, F.Cu at (-240.5, 306.8)
- added TP5: UART Arduino -> PI (3,3V), TestPoint:TestPoint_THTPad_D2.0mm_Drill1.0mm, F.Cu at (-236.5, 302.7)
- added TP6: SDA, TestPoint:TestPoint_THTPad_D2.0mm_Drill1.0mm, F.Cu at (-236.5, 306.8)
- added TP7: SCL, TestPoint:TestPoint_THTPad_D2.0mm_Drill1.0mm, F.Cu at (-232.4, 302.7)
- added TP8: GND(i2c), TestPoint:TestPoint_THTPad_D2.0mm_Drill1.0mm, F.Cu at (-232.4, 306.8)
