File: SmartChessHardware/SmartChessHardware.kicad_pcb (KiCad board)
At the start: 2 copper layers, 294 parts, among them IC1 Pi-Zero-UART, IC2 Arduino_UNO_R3, IC3 MCP23017x-x-SO, J1 Barrel_Jack, SW200 SW_Reed, SW201 SW_Reed, SW202 SW_Reed, SW203 SW_Reed, SW204 SW_Reed, SW205 SW_Reed, SW206 SW_Reed, SW207 SW_Reed, SW208 SW_Reed, SW209 SW_Reed, SW210 SW_Reed, SW211 SW_Reed, SW212 SW_Reed, SW213 SW_Reed, SW214 SW_Reed, SW215 SW_Reed, SW216 SW_Reed, SW217 SW_Reed, SW218 SW_Reed, SW219 SW_Reed, SW220 SW_Reed, SW221 SW_Reed, SW222 SW_Reed, SW223 SW_Reed, SW224 SW_Reed, SW225 SW_Reed, SW226 SW_Reed, SW227 SW_Reed, SW228 SW_Reed, SW229 SW_Reed, SW230 SW_Reed, SW231 SW_Reed, SW232 SW_Reed, SW233 SW_Reed, SW234 SW_Reed, SW235 SW_Reed, SW236 SW_Reed, SW237 SW_Reed, SW238 SW_Reed, SW239 SW_Reed, SW240 SW_Reed, SW241 SW_Reed, SW242 SW_Reed, SW243 SW_Reed, SW244 SW_Reed, SW245 SW_Reed, SW246 SW_Reed, SW247 SW_Reed, SW248 SW_Reed, SW249 SW_Reed, SW250 SW_Reed, SW251 SW_Reed, SW252 SW_Reed, SW253 SW_Reed, SW254 SW_Reed, SW255 SW_Reed, SW256 SW_Reed, SW257 SW_Reed, SW258 SW_Reed, SW259 SW_Reed, SW260 SW_Reed, SW261 SW_Reed, SW262 SW_Reed, SW263 SW_Reed

Commit message: Layout wip
Parts:
- C1: footprint Capacitor_SMD:C_0603_1608Metric -> Capacitor_THT:CP_Radial_D6.3mm_P2.50mm; moved to B.Cu
- C2, C4, F1, IC1, IC2, J1, JP1, JP3, JP4, JP5, R2, R6, TP2: moved to B.Cu
- moved R1 466.5 mm to (114.0, 26.0)
- moved IC1 458.4 mm to (98.2, 42.4), turned to 180 degrees
- moved J1 449.9 mm to (97.3, 31.4)
- moved F1 448.3 mm to (90.5, 23.5), turned to 180 degrees
- moved C4 444.0 mm to (104.0, 45.0)
- moved TP2 440.9 mm to (89.5, 19.0)
- moved C1 437.9 mm to (88.5, 27.3), turned to -90 degrees
- moved TP1 435.6 mm to (86.0, 19.0)
- moved JP1 420.4 mm to (86.0, 23.5), turned to 90 degrees
- moved TP4 420.2 mm to (92.5, 50.5)
- moved R6 418.9 mm to (89.5, 64.7), turned to -90 degrees
- moved R2 416.3 mm to (89.5, 59.2), turned to -90 degrees
- moved TP5 411.8 mm to (92.5, 55.0)
- moved IC3 408.2 mm to (84.0, 113.5)
- moved R4 392.7 mm to (97.5, 121.5), turned to -90 degrees
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Connections:
- IC1 pad 4: (no net) -> +5V
Routing:
- net +5V: track 0.00 -> 646.6 mm, vias 0 -> 4
- net Net-(IC2-D6): track 0.00 -> 141.9 mm
- net Net-(IC1-TX): track 0.00 -> 83.2 mm
- net Net-(JP5-A): track 0.00 -> 65.5 mm
- net Net-(IC2-+5V): track 0.00 -> 52.9 mm
- net Net-(D107-DOUT): track 0.00 -> 43.2 mm
- net Net-(IC3-SCK): track 0.00 -> 27.2 mm
- net Net-(IC3-SDA): track 0.00 -> 26.8 mm
- net Net-(D103-DOUT): track 0.00 -> 26.5 mm
- net Net-(D105-DOUT): track 0.00 -> 26.5 mm
- net Net-(D101-DOUT): track 0.00 -> 26.5 mm
- net Net-(D104-DOUT): track 0.00 -> 26.5 mm
- net Net-(D102-DOUT): track 0.00 -> 26.5 mm
- net Net-(D100-DOUT): track 0.00 -> 26.5 mm
- net Net-(D106-DOUT): track 0.00 -> 26.5 mm
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- added copper zone on B.Cu, net GND
- added copper zone on F.Cu, net GND
Other:
- board outline added: 299 x 243 mm
