File: SmartChessHardware/ScanningMatrix.kicad_sch (KiCad schematic)
At the start: 136 parts, among them SW200 SW_Reed, SW201 SW_Reed, SW202 SW_Reed, SW203 SW_Reed, SW204 SW_Reed, SW205 SW_Reed, SW206 SW_Reed, SW207 SW_Reed, SW208 SW_Reed, SW209 SW_Reed, SW210 SW_Reed, SW211 SW_Reed, SW212 SW_Reed, SW213 SW_Reed, SW214 SW_Reed, SW215 SW_Reed, SW216 SW_Reed, SW217 SW_Reed, SW218 SW_Reed, SW219 SW_Reed, SW220 SW_Reed, SW221 SW_Reed, SW222 SW_Reed, SW223 SW_Reed, SW224 SW_Reed, SW225 SW_Reed, SW226 SW_Reed, SW227 SW_Reed, SW228 SW_Reed, SW229 SW_Reed, SW230 SW_Reed, SW231 SW_Reed, SW232 SW_Reed, SW233 SW_Reed, SW234 SW_Reed, SW235 SW_Reed, SW236 SW_Reed, SW237 SW_Reed, SW238 SW_Reed, SW239 SW_Reed, SW240 SW_Reed, SW241 SW_Reed, SW242 SW_Reed, SW243 SW_Reed, SW244 SW_Reed, SW245 SW_Reed, SW246 SW_Reed, SW247 SW_Reed, SW248 SW_Reed, SW249 SW_Reed, SW250 SW_Reed, SW251 SW_Reed, SW252 SW_Reed, SW253 SW_Reed, SW254 SW_Reed, SW255 SW_Reed, SW256 SW_Reed, SW257 SW_Reed, SW258 SW_Reed, SW259 SW_Reed, SW260 SW_Reed, SW261 SW_Reed, SW262 SW_Reed, SW263 SW_Reed

Commit message: Assigned Footprints
Parts:
- R200, R201, R202, R203, R204, R205, R206, R207: footprint (none) -> Resistor_SMD:R_0603_1608Metric
- SW200, SW201, SW202, SW203, SW204, SW205, SW206, SW207, SW208, SW209, SW210, SW211, SW212, SW213, SW214, SW215, SW216, SW217, SW218, SW219, SW220, SW221, SW222, SW223, SW224, SW225, SW226, SW227, SW228, SW229, SW230, SW231, SW232, SW233, SW234, SW235, SW236, SW237, SW238, SW239, SW240, SW241, SW242, SW243, SW244, SW245, SW246, SW247, SW248, SW249, SW250, SW251, SW252, SW253, SW254, SW255, SW256, SW257, SW258, SW259, SW260, SW261, SW262, SW263: footprint (none) -> Resistor_THT:R_Axial_DIN0309_L9.0mm_D3.2mm_P20.32mm_Horizontal

Commit message: Worked on PCB
Parts:
- D200, D201, D202, D203, D204, D205, D206, D207, D208, D209, D210, D211, D212, D213, D214, D215, D216, D217, D218, D219, D220, D221, D222, D223, D224, D225, D226, D227, D228, D229, D230, D231, D232, D233, D234, D235, D236, D237, D238, D239, D240, D241, D242, D243, D244, D245, D246, D247, D248, D249, D250, D251, D252, D253, D254, D255, D256, D257, D258, D259, D260, D261, D262, D263: footprint Diode_THT:D_DO-41_SOD81_P10.16mm_Horizontal -> Diode_SMD:D_SMA

Commit message: Placed Matrix pull up resistors
Parts:
- renumbered R207 to R200, R200 to R201, R201 to R202, R202 to R203, R203 to R204, R204 to R205, R205 to R206, R206 to R207
Changed lines of the file:
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@@
 		(dnp no)
 		(fields_autoplaced yes)
-		(property "Reference" "R204"
+		(property "Reference" "R205"
 			(at 199.39 34.2899 0)
 			(show_name no)
@@
 			(project "SmartChessHardware"
 				(path "/f14972b6-de47-451d-92ca-2832c545b949/ef711e47-2074-4675-995c-e8c9b46b3f63"
-					(reference "R204")
+					(reference "R205")
 					(unit 1)
 				)
@@
 		(dnp no)
 		(fields_autoplaced yes)
-		(property "Reference" "R203"
+		(property "Reference" "R204"
 			(at 171.45 34.2899 0)
 			(show_name no)
@@
 			(project "SmartChessHardware"
 				(path "/f14972b6-de47-451d-92ca-2832c545b949/ef711e47-2074-4675-995c-e8c9b46b3f63"
-					(reference "R203")
+					(reference "R204")
 					(unit 1)
 				)
@@
 		(dnp no)
 		(fields_autoplaced yes)
-		(property "Reference" "R206"
+		(property "Reference" "R207"
 			(at 256.54 34.2899 0)
 			(show_name no)
@@
 			(project "SmartChessHardware"
 				(path "/f14972b6-de47-451d-92ca-2832c545b949/ef711e47-2074-4675-995c-e8c9b46b3f63"
-					(reference "R206")
+					(reference "R207")
 					(unit 1)
 				)
@@
 		(dnp no)
 		(fields_autoplaced yes)
-		(property "Reference" "R207"
+		(property "Reference" "R200"
 			(at 58.42 35.5599 0)
 			(show_name no)
@@
 			(project "SmartChessHardware"
 				(path "/f14972b6-de47-451d-92ca-2832c545b949/ef711e47-2074-4675-995c-e8c9b46b3f63"
-					(reference "R207")
+					(reference "R200")
 					(unit 1)
 				)
@@
 		(dnp no)
 		(fields_autoplaced yes)
-		(property "Reference" "R202"
+		(property "Reference" "R203"
 			(at 143.51 34.2899 0)
 			(show_name no)
@@
 			(project "SmartChessHardware"
 				(path "/f14972b6-de47-451d-92ca-2832c545b949/ef711e47-2074-4675-995c-e8c9b46b3f63"
-					(reference "R202")
+					(reference "R203")
 					(unit 1)
 				)
@@
 		(dnp no)
 		(fields_autoplaced yes)
-		(property "Reference" "R201"
+		(property "Reference" "R202"
 			(at 115.57 34.2899 0)
 			(show_name no)
@@
 			(project "SmartChessHardware"
 				(path "/f14972b6-de47-451d-92ca-2832c545b949/ef711e47-2074-4675-995c-e8c9b46b3f63"
-					(reference "R201")
+					(reference "R202")
 					(unit 1)
 				)
@@
 		(dnp no)
 		(fields_autoplaced yes)
-		(property "Reference" "R205"
+		(property "Reference" "R206"
 			(at 228.6 34.2899 0)
 			(show_name no)
@@
 			(project "SmartChessHardware"
 				(path "/f14972b6-de47-451d-92ca-2832c545b949/ef711e47-2074-4675-995c-e8c9b46b3f63"
-					(reference "R205")
+					(reference "R206")
 					(unit 1)
 				)
@@
 		(dnp no)
 		(fields_autoplaced yes)
-		(property "Reference" "R200"
+		(property "Reference" "R201"
 			(at 86.36 34.2899 0)
 			(show_name no)
@@
 			(project "SmartChessHardware"
 				(path "/f14972b6-de47-451d-92ca-2832c545b949/ef711e47-2074-4675-995c-e8c9b46b3f63"
-					(reference "R200")
+					(reference "R201")
 					(unit 1)
 				)
